File: kicad/Autobalanced_Photodetector/HV_Regulator_Neg.kicad_sch (KiCad schematic)
At the start: 0 parts

Commit message: feat(kicad): add HV regulators and reference control
Parts:
- added C10, C8, C9: 100n, Capacitor_SMD:C_0805_2012Metric, symbol Device:C
- added C11: 10n, Capacitor_SMD:C_0805_2012Metric, symbol Device:C
- added C12: 3.3u, Capacitor_THT:C_Rect_L29.0mm_W12.2mm_P27.50mm_MKT, symbol Device:C
- added C13: 10n, Capacitor_SMD:C_1206_3216Metric, symbol Device:C
- added D3, D4: MMSZ5242B-E3-08, Diode_SMD:D_SOD-123, symbol Device:D_Zener
- added Q3, Q4: TP2540N8-G, Package_TO_SOT_SMD:SOT-89-3, symbol Device:Q_PMOS_GDS
- added R19: 1k, Resistor_SMD:R_0805_2012Metric, symbol Device:R
- added R20, R22: 470k, Resistor_SMD:R_1206_3216Metric, symbol Device:R
- added R21, R25: 10k, Resistor_SMD:R_0805_2012Metric, symbol Device:R
- added R23: 10, Resistor_SMD:R_0805_2012Metric, symbol Device:R
- added R24: 47k, Resistor_SMD:R_0805_2012Metric, symbol Device:R
- added R26, R28: 1.1k, Resistor_SMD:R_0805_2012Metric, symbol Device:R
- added R27: 100k, Resistor_SMD:R_0805_2012Metric, symbol Device:R
- added U4: OPA2192ID, Package_SO:SOIC-8_3.9x4.9mm_P1.27mm, symbol Amplifier_Operational:LM358
Connections:
- new net: R24.1, U4.1, U4.5 (+)
- new net: D3.1 (K), Q3.3 (S), R21.1, U4.6 (-)
- new net: R19.1, U4.7
- new net: D4.2 (A), Q3.2 (D), Q4.1 (G), R20.2, R22.2
- new net: Q4.2 (D), R23.2
- new net: D3.2 (A), Q3.1 (G), R19.2
- new net: R26.2, R27.1, U4.3 (+)
- new net: C11.1, R24.2
- new net: C11.2, R25.1, U4.2 (-)
- new net: R26.1, R28.2
- new net AGND: C10.2, C12.2, C13.2, C9.2, R27.2
- new net HV_BIAS_NEG: C12.1, C13.1, D4.1 (K), Q4.3 (S), R28.1
- new net HV_RAW_NEG: R20.1, R22.1, R23.1
- new net VCC_12V: C8.2, C9.1, R21.2, U4.8 (V+)
- new net VEE_12V: C10.1, C8.1, U4.4 (V-)
- new net V_REF_NEG: R25.2
